Commit message: adjust tool rpy

File: urdf/rccn_west_robot_with_tool.urdf (robot description, URDF)
Before this commit: robot rccn_west_robot_with_tool, 14 links, 13 joints
Joints:
- joint tcp_joint: origin xyz=0 0 0.36 rpy=0 0 0 -> xyz=0 0 0.36 rpy=-3.14159265 0 -3.14159265

File: urdf/tool.xacro (robot description, xacro)
@@ -27,5 +27,5 @@
     <!-- TCP frame -->
     <joint name="${prefix}tcp_joint" type="fixed">
-      <origin xyz="0 0 0.36" rpy="0 0 0"/>
+      <origin xyz="0 0 0.36" rpy="-3.14159265 0 -3.14159265"/>
       <parent link="${prefix}tool"/>
       <child link="${prefix}tcp"/>
